File: hardware/driver.kicad_pcb (KiCad board)
At the start: 2 copper layers, 24 x 23 mm, 20 parts, among them Q1 BSS84, Q2 BSS138, Q3 BSS138, Q4 BSS84, Q5 BSS138, Q6 BSS138

Commit message: Annotation completed
Other:
- board text added: "CC BY-SA"
- board text added: "Rev 1.0"
- board text added: "©2017 Paul Qureshi"
Changed lines of the file:
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@@
 (kicad_pcb (version 4) (host pcbnew 4.0.5)
   (general
-    (links 0)
-    (no_connects 7)
+    (links 27)
+    (no_connects 0)
     (area 99.924999 56.924999 124.075001 80.075001)
     (thickness 1.6)
-    (drawings 85)
+    (drawings 90)
     (tracks 87)
     (zones 0)
@@
     (34 B.Paste user)
     (35 F.Paste user)
-    (36 B.SilkS user)
-    (37 F.SilkS user)
+    (36 B.SilkS user hide)
+    (37 F.SilkS user hide)
     (38 B.Mask user)
     (39 F.Mask user)
@@
     (45 Margin user)
     (46 B.CrtYd user)
-    (47 F.CrtYd user)
+    (47 F.CrtYd user hide)
     (48 B.Fab user)
-    (49 F.Fab user)
+    (49 F.Fab user hide)
   )
   (setup
@@
     (pad_to_mask_clearance 0.2)
     (aux_axis_origin 0 0)
-    (visible_elements FFFEFF7F)
+    (visible_elements FFFCFB7F)
     (pcbplotparams
       (layerselection 0x00030_80000001)
@@
       (xy -2.796116 -1.725084) (xy -2.797198 -2.094474) (xy -2.798279 -2.463863) (xy -0.037064 -2.46272)) (layer Eco2.User) (width 0.01))
   )
+  (gr_text "Rev 1.0" (at 104 72) (layer Eco2.User)
+    (effects (font (size 1 1) (thickness 0.2)) (justify mirror))
+  )
+  (gr_text "CC BY-SA" (at 112 59) (layer Eco2.User)
+    (effects (font (size 1 1) (thickness 0.2)) (justify mirror))
+  )
+  (gr_text "©2017 Paul Qureshi" (at 122.8 64.7 90) (layer B.Cu)
+    (effects (font (size 0.9 0.9) (thickness 0.125)) (justify mirror))
+  )
+  (dimension 23 (width 0.3) (layer Eco1.User)
+    (gr_text "23.000 mm" (at 127.35 68.5 270) (layer Eco1.User)
+      (effects (font (size 1.5 1.5) (thickness 0.3)))
+    )
+    (feature1 (pts (xy 125 80) (xy 128.7 80)))
+    (feature2 (pts (xy 125 57) (xy 128.7 57)))
+    (crossbar (pts (xy 126 57) (xy 126 80)))
+    (arrow1a (pts (xy 126 80) (xy 125.413579 78.873496)))
+    (arrow1b (pts (xy 126 80) (xy 126.586421 78.873496)))
+    (arrow2a (pts (xy 126 57) (xy 125.413579 58.126504)))
+    (arrow2b (pts (xy 126 57) (xy 126.586421 58.126504)))
+  )
+  (dimension 24 (width 0.3) (layer Eco1.User)
+    (gr_text "24.000 mm" (at 112 53.65) (layer Eco1.User)
+      (effects (font (size 1.5 1.5) (thickness 0.3)))
+    )
+    (feature1 (pts (xy 124 56) (xy 124 52.3)))
+    (feature2 (pts (xy 100 56) (xy 100 52.3)))
+    (crossbar (pts (xy 100 55) (xy 124 55)))
+    (arrow1a (pts (xy 124 55) (xy 122.873496 55.586421)))
+    (arrow1b (pts (xy 124 55) (xy 122.873496 54.413579)))
+    (arrow2a (pts (xy 100 55) (xy 101.126504 55.586421)))
+    (arrow2b (pts (xy 100 55) (xy 101.126504 54.413579)))
+  )
   (gr_line (start 113.1 67.9) (end 113.1 68.7) (layer Eco1.User) (width 0.2))
