File: hardware/driver.kicad_pcb (KiCad board)
At the start: 2 copper layers, 24 x 23 mm, 20 parts, among them Q1 BSS84, Q2 BSS138, Q3 BSS138, Q4 BSS84, Q5 BSS138, Q6 BSS138

Commit message: DRC, output
Routing:
- net GND: track 14.8 -> 15.4 mm
Changed lines of the file:
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@@
     (links 27)
     (no_connects 0)
-    (area 99.924999 56.924999 124.075001 80.075001)
+    (area 99.924999 52.3 133.85 81.5274)
     (thickness 1.6)
     (drawings 90)
-    (tracks 87)
+    (tracks 88)
     (zones 0)
     (modules 20)
@@
     (40 Dwgs.User user)
     (41 Cmts.User user)
-    (42 Eco1.User user)
-    (43 Eco2.User user hide)
+    (42 Eco1.User user hide)
+    (43 Eco2.User user)
     (44 Edge.Cuts user)
     (45 Margin user)
@@
     (visible_elements FFFCFB7F)
     (pcbplotparams
-      (layerselection 0x00030_80000001)
-      (usegerberextensions false)
+      (layerselection 0x01ccc_80000001)
+      (usegerberextensions true)
       (excludeedgelayer true)
       (linewidth 0.100000)
@@
       (plotinvisibletext false)
       (padsonsilk false)
-      (subtractmaskfromsilk false)
+      (subtractmaskfromsilk true)
       (outputformat 1)
       (mirror false)
-      (drillshape 1)
+      (drillshape 0)
       (scaleselection 1)
-      (outputdirectory ""))
+      (outputdirectory plot/))
   )
   (net 0 "")
@@
       (xy -2.796116 -1.725084) (xy -2.797198 -2.094474) (xy -2.798279 -2.463863) (xy -0.037064 -2.46272)) (layer Eco2.User) (width 0.01))
   )
-  (gr_text "Rev 1.0" (at 104 72) (layer Eco2.User)
+  (gr_text "Rev 1.0" (at 112 72.5) (layer Eco2.User)
     (effects (font (size 1 1) (thickness 0.2)) (justify mirror))
   )
@@
     (effects (font (size 0.9 0.9) (thickness 0.125)) (justify mirror))
   )
-  (dimension 23 (width 0.3) (layer Eco1.User)
-    (gr_text "23.000 mm" (at 127.35 68.5 270) (layer Eco1.User)
+  (dimension 23 (width 0.3) (layer Dwgs.User)
+    (gr_text "23.000 mm" (at 127.35 68.5 270) (layer Dwgs.User)
       (effects (font (size 1.5 1.5) (thickness 0.3)))
     )
@@
     (arrow2b (pts (xy 126 57) (xy 126.586421 58.126504)))
   )
-  (dimension 24 (width 0.3) (layer Eco1.User)
-    (gr_text "24.000 mm" (at 112 53.65) (layer Eco1.User)
+  (dimension 24 (width 0.3) (layer Dwgs.User)
+    (gr_text "24.000 mm" (at 112 53.65) (layer Dwgs.User)
       (effects (font (size 1.5 1.5) (thickness 0.3)))
     )
@@
   (via (at 107.7 73.3) (size 0.6) (drill 0.4) (layers F.Cu B.Cu) (net 4))
   (segment (start 111 74) (end 111 77) (width 0.75) (layer F.Cu) (net 4))
+  (segment (start 120.95 66) (end 120.95 65.05) (width 1) (layer F.Cu) (net 5))
+  (segment (start 120.95 65.05) (end 121 65) (width 1) (layer F.Cu) (net 5))
+  (via (at 121 65) (size 0.6) (drill 0.4) (layers F.Cu B.Cu) (net 5))
+  (segment (start 109.95 66) (end 109.95 67.95) (width 1) (layer F.Cu) (net 5))
+  (segment (start 109.95 67.95) (end 110 68) (width 1) (layer F.Cu) (net 5))
+  (via (at 110 68) (size 0.6) (drill 0.4) (layers F.Cu B.Cu) (net 5))
   (segment (start 110 61) (end 111.1 61) (width 1) (layer F.Cu) (net 5))
   (via (at 111.1 61) (size 0.6) (drill 0.4) (layers F.Cu B.Cu) (net 5))
@@
   (segment (start 118.95 72.15) (end 119 72.2) (width 1) (layer F.Cu) (net 5))
   (via (at 119 72.2) (size 0.6) (drill 0.4) (layers F.Cu B.Cu) (net 5))
-  (segment (start 120.95 66) (end 122.2 66) (width 1) (layer F.Cu) (net 5))
-  (via (at 122.2 66) (size 0.6) (drill 0.4) (layers F.Cu B.Cu) (net 5))
   (segment (start 120.95 66) (end 120.95 67.15) (width 1) (layer F.Cu) (net 5))
   (segment (start 120.95 67.15) (end 121 67.2) (width 1) (layer F.Cu) (net 5))
@@
   (segment (start 109.95 66) (end 111.2 66) (width 1) (layer F.Cu) (net 5))
   (via (at 111.2 66) (size 0.6) (drill 0.4) (layers F.Cu B.Cu) (net 5))
-  (segment (start 109.95 66) (end 109.95 67.15) (width 1) (layer F.Cu) (net 5))
-  (segment (start 109.95 67.15) (end 110 67.2) (width 1) (layer F.Cu) (net 5))
-  (via (at 110 67.2) (size 0.6) (drill 0.4) (layers F.Cu B.Cu) (net 5))
   (segment (start 103 73.8) (end 104 73.8) (width 1) (layer F.Cu) (net 5))
   (via (at 104 73.8) (size 0.6) (drill 0.4) (layers F.Cu B.Cu) (net 5))
